File: module_pcb_thermal_mockup_v3.5/design-files/module_pcb_thermal_mockup_v3.5/module_pcb_thermal_mockup_v3.5.kicad_pcb (KiCad board)
At the start: 4 copper layers, 44.1 x 57.5 mm, 55 parts, among them J1 Conn_02x06_Counter_Clockwise, U1 ETROC_dummy_thermal_sensors, U2 ETROC_dummy_thermal_sensors, U3 ETROC_dummy_thermal_sensors, U4 ETROC_dummy_thermal_sensors, U5 AD77x8, U6 AD780, U7 TMP121, U8 TMP121, U9 TMP121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

Commit message: cleaned up DRC
Routing:
- net GND: track 73.6 -> 88.4 mm, vias 32 -> 33
- net +5V: track 50.9 -> 63.9 mm, vias 18 -> 24
- net /DOUT: track 95.2 -> 98.2 mm, vias 5 -> 6
- net /CS_T3: track 32.7 -> 35.0 mm
- net VCC: track 162.0 -> 163.8 mm
- net /DIN: track 25.4 -> 26.7 mm
- net /CS: track 34.8 -> 33.6 mm
- net /ETROC2: track 69.9 -> 71.0 mm
- net /CLK: track 110.6 -> 110.3 mm, vias 5 -> 6
Other:
- board text added: "DIN ~{RST} +5V ~{CS_T2} CLK GND"
- board text added: "~{CS} ~{RDY} DOUT ~{CS_T1} VCC ~{CS_T3}"
- board text removed: "CS ~{RDY} DOUT CS_T1 VCC CS_T3"
- board text removed: "DIN ~{RST} +5V CS_T2 CLK GND"
