File: control-board/control-board_v1/control-board_v1-p2.kicad_sch (KiCad schematic)
At the start: 20 parts, among them Q10 NMOS, Q9 NMOS, U3 ADS1118, U4 Opamp_Dual, U6 Opamp_Dual

Commit message: pcb design change
Connections:
- net 1-Heater: no longer R28.2, U4.3 (+)
- net 2-Heater: no longer R28.2, U4.5 (+)
- net 3-Heater: no longer R28.2, U6.3 (+)
- net 4-Heater: no longer R28.2, U6.5 (+)
- new net 1-GND: R28.2, U4.3 (+)
- new net 2-GND: R28.2, U4.5 (+)
- new net 3-GND: R28.2, U6.3 (+)
- new net 4-GND: R28.2, U6.5 (+)
Other:
- moved on the sheet: R28
