File: module_pcb_thermal_mockup_v4/design-files/module_pcb_thermal_mockup_v4/module_pcb_thermal_mockup_v4.kicad_sch (KiCad schematic)
At the start: 49 parts, among them J1 Conn_02x06_Counter_Clockwise, U1 ETROC_dummy_thermal_sensors, U2 ETROC_dummy_thermal_sensors, U3 ETROC_dummy_thermal_sensors, U4 ETROC_dummy_thermal_sensors, U5 AD77x8, U6 AD780, U7 TMP121, U8 TMP121, U9 TMP121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

Commit message: bumpbond measurement
Parts:
- removed BumpBonds1: TestPoint, TestPoint:TestPoint_Pad_1.0x1.0mm, symbol Connector:TestPoint
- removed JMPR2: 0, Resistor_SMD:R_0805_2012Metric_Pad1.20x1.40mm_HandSolder, symbol Device:R
- added TP+1, TP-1, TP-2, TP-3, TP-4: TestPoint, TestPoint:TestPoint_Pad_1.0x1.0mm, symbol Connector:TestPoint
Connections:
- net VCC: no longer U1.1 (VCC), U2.1 (VCC), U3.121 (VSS), U4.121 (VSS)
- net VSS renamed TP+
- net TP+: now also U1.1 (VCC), U2.1 (VCC), TP+1.1; no longer U1.121 (VSS), U2.121 (VSS)
- new net: TP-2.1, U2.121 (VSS)
- new net: TP-3.1, U3.121 (VSS)
- new net: TP-4.1, U4.121 (VSS)
- new net: TP-1.1, U1.121 (VSS)
