File: module_pcb_thermal_mockup_v4/design-files/module_pcb_thermal_mockup_v4/module_pcb_thermal_mockup_v4.kicad_pcb (KiCad board)
At the start: 4 copper layers, 44.1 x 57.5 mm, 56 parts, among them J1 Conn_02x06_Counter_Clockwise, U1 ETROC_dummy_thermal_sensors, U2 ETROC_dummy_thermal_sensors, U3 ETROC_dummy_thermal_sensors, U4 ETROC_dummy_thermal_sensors, U5 AD77x8, U6 AD780, U7 TMP121, U8 TMP121, U9 TMP121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

Commit message: bumpbond measurement
Parts:
- removed JMPR2: 0, Resistor_SMD:R_0805_2012Metric_Pad1.20x1.40mm_HandSolder
- removed R-Bonds: TestPoint, TestPoint:TestPoint_Pad_1.0x1.0mm
- added TP+: TestPoint, TestPoint:TestPoint_Pad_1.0x1.0mm, B.Cu at (41.0, 28.8)
- added TP-1: TestPoint, TestPoint:TestPoint_Pad_1.0x1.0mm, B.Cu at (19.6, 51.2)
- added TP-2: TestPoint, TestPoint:TestPoint_Pad_1.0x1.0mm, B.Cu at (42.0, 44.5)
- added TP-3: TestPoint, TestPoint:TestPoint_Pad_1.0x1.0mm, B.Cu at (3.00, 4.70)
- added TP-4: TestPoint, TestPoint:TestPoint_Pad_1.0x1.0mm, B.Cu at (22.0, 5.20)
- moved VCC 24.9 mm to (31.9, 31.0), turned to 0 degrees
- renumbered VCC1 to VCC
Connections:
- U1 pad 1: VCC -> TP+
- U1 pad 121: /VSS -> Net-(U1-VSS)
- U2 pad 1: VCC -> TP+
- U2 pad 121: /VSS -> Net-(U2-VSS)
- U3 pad 1: /VSS -> TP+
- U3 pad 121: VCC -> Net-(U3-VSS)
- U4 pad 1: /VSS -> TP+
- U4 pad 121: VCC -> Net-(U4-VSS)
Routing:
- net /VSS: track 106.2 -> 0.00 mm, vias 3 -> 0
- net VCC: track 163.8 -> 68.5 mm, vias 5 -> 4
- net TP+: track 0.00 -> 55.7 mm, vias 0 -> 2
- net Net-(U2-VSS): track 0.00 -> 9.35 mm, vias 0 -> 1
- net Net-(U1-VSS): track 0.00 -> 3.18 mm, vias 0 -> 1
- net Net-(U3-VSS): track 0.00 -> 2.84 mm, vias 0 -> 1
- net Net-(U4-VSS): track 0.00 -> 2.18 mm, vias 0 -> 1
- net GND: track 88.4 -> 87.1 mm, vias 33 -> 32
Other:
- board text added: "locked"
- board text removed: "ETL Module PCB Thermal Mockup V4 Boston University N. Gonzalez 07-2024"

Commit message: control board v2
Other:
- board text added: "Fill JMPR1 for PCB heating"
- board text removed: "Fill JMPR1 for PCB heating Fill JMPR2 for chip heating"
Changed lines of the file:
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@@
     (effects (font (size 1 1) (thickness 0.15)) (justify mirror))
   )
-  (gr_text "Fill JMPR1 for PCB heating\nFill JMPR2 for chip heating" (at 1.89 38.29 90) (layer "B.SilkS")
+  (gr_text "Fill JMPR1 for PCB heating\n" (at 1.21 38.25 90) (layer "B.SilkS")
     (effects (font (size 0.8 0.8) (thickness 0.15)) (justify mirror))
   )
