File: control-board/control-board_v2/control-board_v2.kicad_sch (KiCad schematic)
At the start: 17 parts, among them J1 Barrel_Jack, J2 Header-M_2x6, J3 Header-M_2x6, J4 Header-M_2x6, J5 Header-M_2x6, J6 Header_1x8, J7 Header_1x8, J8 Header_1x10, J9 Header_1x8, U1 CD74HCT154M

Commit message: control board v2
Connections:
- net 1-GND is gone; now on net GND: J3.12 (Pin_12)
- net 2-GND is gone; now on net GND: J2.12 (Pin_12)
- net 3-GND is gone; now on net GND: J4.12 (Pin_12)
- net 4-GND is gone; now on net GND: J5.12 (Pin_12)
- net H1-D12 renamed H2-D12
- net H2-D13 renamed H1-D13
Changed lines of the file:
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@@
+    (stroke (width 0) (type default))
+  )
+  (wire (pts (xy 169.9006 83.82) (xy 155.702 83.82))
     (stroke (width 0) (type default))
   )
@@
     (stroke (width 0) (type default))
   )
+  (wire (pts (xy 169.9006 61.341) (xy 155.702 61.341))
+    (stroke (width 0) (type default))
+  )
   (wire (pts (xy 54.483 51.943) (xy 56.388 51.943))
     (stroke (width 0) (type default))
@@
     (stroke (width 0) (type default))
   )
+  (wire (pts (xy 170.0276 106.299) (xy 155.829 106.299))
+    (stroke (width 0) (type default))
+  )
   (wire (pts (xy 230.251 102.743) (xy 230.251 100.203))
+    (stroke (width 0) (type default))
+  )
+  (wire (pts (xy 155.956 128.27) (xy 170.18 128.27))
     (stroke (width 0) (type default))
   )
@@
     )
   )
-  (global_label "1-GND" (shape input) (at 155.702 61.341 0) (fields_autoplaced)
-    (effects (font (size 1.27 1.27)) (justify left))
-    (property "Intersheetrefs" "${INTERSHEET_REFS}" (at 165.3396 61.341 0)
-      (effects (font (size 1.27 1.27)) (justify left) hide)
-    )
-  )
   (global_label "2-CS_T2" (shape input) (at 155.702 93.98 0) (fields_autoplaced)
     (effects (font (size 1.27 1.27)) (justify left))
@@
     )
   )
-  (global_label "4-GND" (shape input) (at 155.956 128.27 0) (fields_autoplaced)
-    (effects (font (size 1.27 1.27)) (justify left))
-    (property "Intersheetrefs" "${INTERSHEET_REFS}" (at 165.5936 128.27 0)
-      (effects (font (size 1.27 1.27)) (justify left) hide)
-    )
-  )
   (global_label "1-CS" (shape input) (at 71.628 50.673 0) (fields_autoplaced)
     (effects (font (size 1.27 1.27)) (justify left))
@@
     )
   )
-  (global_label "H1-D12" (shape input) (at 243.586 87.503 180) (fields_autoplaced)
+  (global_label "H2-D12" (shape input) (at 243.586 87.503 180) (fields_autoplaced)
     (effects (font (size 1.27 1.27)) (justify right))
     (property "Intersheetrefs" "${INTERSHEET_REFS}" (at 232.7994 87.503 0)
@@
     )
   )
-  (global_label "H2-D13" (shape input) (at 243.586 90.043 180) (fields_autoplaced)
+  (global_label "H1-D13" (shape input) (at 243.586 90.043 180) (fields_autoplaced)
     (effects (font (size 1.27 1.27)) (justify right))
     (property "Intersheetrefs" "${INTERSHEET_REFS}" (at 232.7994 90.043 0)
@@
     )
   )
-  (global_label "3-GND" (shape input) (at 155.829 106.299 0) (fields_autoplaced)
-    (effects (font (size 1.27 1.27)) (justify left))
-    (property "Intersheetrefs" "${INTERSHEET_REFS}" (at 165.4666 106.299 0)
-      (effects (font (size 1.27 1.27)) (justify left) hide)
-    )
-  )
   (global_label "1-CS_T2" (shape input) (at 155.702 71.501 0) (fields_autoplaced)
     (effects (font (size 1.27 1.27)) (justify left))
@@
     (effects (font (size 1.27 1.27)) (justify left))
     (property "Intersheetrefs" "${INTERSHEET_REFS}" (at 83.0193 65.913 0)
-      (effects (font (size 1.27 1.27)) (justify left) hide)
-    )
-  )
-  (global_label "2-GND" (shape input) (at 155.702 83.82 0) (fields_autoplaced)
-    (effects (font (size 1.27 1.27)) (justify left))
-    (property "Intersheetrefs" "${INTERSHEET_REFS}" (at 165.3396 83.82 0)
       (effects (font (size 1.27 1.27)) (justify left) hide)
     )
@@
         (path "/5ea0e920-d127-456d-9ad4-df9bbc649b9b"
           (reference "#PWR040") (unit 1)
+        )
+      )
+    )
+  )
+  (symbol (lib_id "power:GND") (at 169.9006 61.341 0) (unit 1)
+    (in_bom yes) (on_board yes) (dnp no)
+    (property "Reference" "#PWR08" (at 169.9006 67.691 0)
+      (effects (font (size 1.27 1.27)) hide)
+    )
+    (property "Value" "GND" (at 169.9006 65.151 0)
+      (effects (font (size 1.27 1.27)))
+    )
+    (property "Footprint" "" (at 169.9006 61.341 0)
+      (effects (font (size 1.27 1.27)) hide)
+    )
+    (property "Datasheet" "" (at 169.9006 61.341 0)
+      (effects (font (size 1.27 1.27)) hide)
+    )
+    (pin "1")
+    (instances
+      (project "control-board_v2"
+        (path "/5ea0e920-d127-456d-9ad4-df9bbc649b9b"
+          (reference "#PWR08") (unit 1)
+        )
+      )
+      (project "arduino_uno"
+        (path "/b1128066-0aeb-425d-915d-968e839977c3"
+          (reference "#PWR046") (unit 1)
         )
       )
@@
     )
   )
+  (symbol (lib_id "power:GND") (at 169.9006 83.82 0) (unit 1)
+    (in_bom yes) (on_board yes) (dnp no)
+    (property "Reference" "#PWR012" (at 169.9006 90.17 0)
+      (effects (font (size 1.27 1.27)) hide)
+    )
+    (property "Value" "GND" (at 169.9006 87.63 0)
+      (effects (font (size 1.27 1.27)))
+    )
+    (property "Footprint" "" (at 169.9006 83.82 0)
+      (effects (font (size 1.27 1.27)) hide)
+    )
+    (property "Datasheet" "" (at 169.9006 83.82 0)
+      (effects (font (size 1.27 1.27)) hide)
+    )
+    (pin "1")
+    (instances
+      (project "control-board_v2"
+        (path "/5ea0e920-d127-456d-9ad4-df9bbc649b9b"
+          (reference "#PWR012") (unit 1)
+        )
+      )
+      (project "arduino_uno"
+        (path "/b1128066-0aeb-425d-915d-968e839977c3"
+          (reference "#PWR046") (unit 1)
+        )
+      )
+    )
+  )
   (symbol (lib_id "power:+5V") (at 54.483 51.181 0) (unit 1)
     (in_bom yes) (on_board yes) (dnp no) (fields_autoplaced)
@@
     )
   )
+  (symbol (lib_id "power:GND") (at 170.18 128.27 0) (unit 1)
+    (in_bom yes) (on_board yes) (dnp no)
+    (property "Reference" "#PWR019" (at 170.18 134.62 0)
+      (effects (font (size 1.27 1.27)) hide)
+    )
+    (property "Value" "GND" (at 170.18 132.08 0)
+      (effects (font (size 1.27 1.27)))
+    )
+    (property "Footprint" "" (at 170.18 128.27 0)
+      (effects (font (size 1.27 1.27)) hide)
+    )
+    (property "Datasheet" "" (at 170.18 128.27 0)
+      (effects (font (size 1.27 1.27)) hide)
+    )
+    (pin "1")
+    (instances
+      (project "control-board_v2"
+        (path "/5ea0e920-d127-456d-9ad4-df9bbc649b9b"
+          (reference "#PWR019") (unit 1)
+        )
+      )
+      (project "arduino_uno"
+        (path "/b1128066-0aeb-425d-915d-968e839977c3"
+          (reference "#PWR046") (unit 1)
+        )
+      )
+    )
+  )
   (symbol (lib_id "Device:C_Polarized") (at 253.492 42.799 0) (unit 1)
     (in_bom yes) (on_board yes) (dnp no) (fields_autoplaced)
@@
         )
       )
+    )
+  )
+  (symbol (lib_id "power:GND") (at 170.0276 106.299 0) (unit 1)
+    (in_bom yes) (on_board yes) (dnp no)
+    (property "Reference" "#PWR016" (at 170.0276 112.649 0)
+      (effects (font (size 1.27 1.27)) hide)
+    )
+    (property "Value" "GND" (at 170.0276 110.109 0)
+      (effects (font (size 1.27 1.27)))
+    )
+    (property "Footprint" "" (at 170.0276 106.299 0)
+      (effects (font (size 1.27 1.27)) hide)
+    )
+    (property "Datasheet" "" (at 170.0276 106.299 0)
+      (effects (font (size 1.27 1.27)) hide)
+    )
+    (pin "1")
+    (instances
+      (project "control-board_v2"
+        (path "/5ea0e920-d127-456d-9ad4-df9bbc649b9b"
+          (reference "#PWR016") (unit 1)
+        )
+      )
+      (project "arduino_uno"
+        (path "/b1128066-0aeb-425d-915d-968e839977c3"
+          (reference "#PWR046") (unit 1)
+        )
+      )
