File: control-board/control-board_v2/control-board_v2-p2.kicad_sch (KiCad schematic)
At the start: 40 parts, among them Q1 NMOS, Q2 NMOS, Q3 NMOS, Q9 NMOS, U2 Opamp_Dual, U3 ADS1118, U4 Opamp_Dual, U5 Opamp_Dual, U6 Opamp_Dual

Commit message: control board v2
Parts:
- removed R28 (x4): 20K, Resistor_SMD:R_0805_2012Metric, symbol Device:R_Small_US
- removed R28 (x4): 10K, Resistor_SMD:R_0805_2012Metric, symbol Device:R_Small_US
- removed U5, U6: Opamp_Dual, Package_SO:SOIC-8_3.9x4.9mm_P1.27mm, symbol Device:Opamp_Dual
- added R28: 20K, Resistor_SMD:R_0805_2012Metric, symbol Device:R_Small_US
- added R28: 10K, Resistor_SMD:R_0805_2012Metric, symbol Device:R_Small_US
- added unit 2 of U2
- added unit 3 of U2
- added unit 2 of U4
- U2, U4: PartNum MCP6487T-E/SN -> (none)
- renumbered Q9 to Q1, Q3 to Q2
Connections:
- net +5V: now also U2.8 (V+)
- net +9V: now also R28.2
- net GND: now also Q1.2 (S), Q2.2 (S), R28.2, U2.4 (V-); no longer Q1.5 (S), Q2.5 (S)
- net H3-D18: now also Q2.3 (G); no longer Q2.1 (G)
- net V_{h1}: now also U2.1; no longer U4.1
- net V_{h2}: now also U2.7; no longer U2.1
- net V_{h3}: now also U4.1
- net V_{h4}: now also U4.7
- net Com-Node: now reaches U4.3 (+)
- net Com-Node: now also U2.3 (+), R28.1, R28.1, U2.5 (+), U4.5 (+)
- net 1-Heater: now reaches Q1.6 (D), R28.1, R28.2
- net at R28.1, R28.2: now also U2.6 (-); no longer U2.2 (-)
- net at R28.1, R28.2: now also U2.2 (-); no longer U4.2 (-)
- net at R28.1, R28.2: now also U4.6 (-)
- net 2-Heater: now reaches R28.1, R28.2
- net 2-Heater: now also Q1.4 (D); no longer Q1.6 (D)
- net 4-Heater: now reaches Q2.6 (D), R28.1, R28.2
- net at R28.1, R28.2: now also U4.2 (-)
- net 3-Heater: now reaches R28.1, R28.2
- net 3-Heater: now also Q2.4 (D); no longer Q2.6 (D)
- net H1-D12 renamed H1-D13
- removed net H2-D13: Q1.1 (G)
- new net H2-D12: Q1.3 (G)

Commit message: v3 with relay
Parts:
- removed Q1, Q2: NMOS, Package_TO_SOT_SMD:SOT-23-6, symbol Device:Q_Dual_NMOS_G1S2G2D2S1D1
- removed R28 (x5): 20K, Resistor_SMD:R_0805_2012Metric, symbol Device:R_Small_US
- removed R28 (x3): 100, Resistor_SMD:R_0805_2012Metric, symbol Device:R_Small_US
- removed R28 (x4): 0.003, Resistor_SMD:R_2512_6332Metric, symbol Device:R_Small_US
- removed R28 (x5): 10K, Resistor_SMD:R_0805_2012Metric, symbol Device:R_Small_US
- removed R28 (x3): 166K, Resistor_SMD:R_0603_1608Metric, symbol Device:R_Small_US
- added R28 (x7): 100, Resistor_SMD:R_0805_2012Metric, symbol Device:R_Small_US
- added R28 (x7): 166K, Resistor_SMD:R_0805_2012Metric, symbol Device:R_Small_US
- added R28 (x4): 0.003, Resistor_SMD:R_2512_6332Metric, symbol Device:R_Small_US
- added U5, U6, U8, U9: LCA701STR, Package_SO:SOIC-6_New, symbol Relay_SolidState:TLP148G
- R28: footprint Resistor_SMD:R_0603_1608Metric -> Resistor_SMD:R_0805_2012Metric
- U2, U4: Part (none) -> LM358DR
Connections:
- net +5V: no longer C3.1, C7.1, U2.8 (V+), U4.8 (V+)
- net +9V: now also C3.1, C7.1, U2.8 (V+), U4.8 (V+), U5.4, U5.6, U6.4, U6.6, U8.4, U8.6, U9.4, U9.6
- net 1-Heater: now also R28.1, R28.2
- net 2-Heater: now also R28.1, R28.2
- net 3-Heater: now also R28.1, R28.2
- net 4-Heater: now also R28.1, R28.2
- net GND: now also R28.2, R28.2, R28.2, R28.2, U5.3, U6.3, U8.3, U9.3
- net H1-D13: now also U6.1
- net H2-D12: now also U5.1
- net H3-D18: now also U8.1
- net H4-D19: now also U9.1
- net V_{h1}: now also R28.1; no longer R28.1
- net V_{h2}: now also R28.1
- net V_{h3}: now also R28.1
- net V_{h4}: now also R28.1
- net at R28.2: now also R28.1, U6.5
- net at U2.6 (-): now also R28.2, R28.2
- net at U4.6 (-): now also R28.2, R28.2
- net at U4.2 (-): now also R28.2, R28.2
- removed net Com-Node: U2.3 (+), U2.5 (+), U4.3 (+), U4.5 (+)
- new net: R28.1, R28.1, U4.3 (+)
- new net: R28.1, R28.2, U8.5
- new net: R28.1, R28.1, U2.5 (+)
- new net: R28.1, R28.2, U5.5
- new net: R28.1, R28.1, U4.5 (+)
- new net: R28.1, R28.1, U2.3 (+)
- new net: R28.2, R28.2, U2.2 (-)
- new net: R28.1, R28.2, U9.5
Other:
- note removed: "G = 1+ R22/R21 G = 1 + 166k/100 G = 1661"
- moved on the sheet: C3, C7, R28, U2A, U2C, U4C

Commit message: final layout for controlboard v3
Connections:
- net GND: now also U5.2, U6.2, U8.2, U9.2; no longer U5.3, U6.3, U8.3, U9.3
Changed lines of the file:
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@@
     )
     (pin "1")
-    (pin "3")
+    (pin "2")
     (pin "4")
     (pin "5")
@@
     )
   )
-  (symbol (lib_id "Relay_SolidState:TLP148G") (at 84.836 130.937 0) (unit 1)
+  (symbol (lib_name "TLP148G_3") (lib_id "Relay_SolidState:TLP148G") (at 84.836 130.937 0) (unit 1)
     (in_bom yes) (on_board yes) (dnp no) (fields_autoplaced)
     (property "Reference" "U8" (at 84.836 122.3772 0)
@@
     )
     (pin "1")
-    (pin "3")
+    (pin "2")
     (pin "4")
     (pin "5")
@@
     )
   )
-  (symbol (lib_id "Relay_SolidState:TLP148G") (at 84.6582 94.4118 0) (unit 1)
+  (symbol (lib_name "TLP148G_2") (lib_id "Relay_SolidState:TLP148G") (at 84.6582 94.4118 0) (unit 1)
     (in_bom yes) (on_board yes) (dnp no) (fields_autoplaced)
     (property "Reference" "U5" (at 84.6582 85.852 0)
@@
     )
     (pin "1")
-    (pin "3")
+    (pin "2")
     (pin "4")
     (pin "5")
@@
     )
   )
-  (symbol (lib_id "Relay_SolidState:TLP148G") (at 85.1662 54.5846 0) (unit 1)
+  (symbol (lib_name "TLP148G_1") (lib_id "Relay_SolidState:TLP148G") (at 85.1662 54.5846 0) (unit 1)
     (in_bom yes) (on_board yes) (dnp no) (fields_autoplaced)
     (property "Reference" "U6" (at 85.1662 46.0248 0)
@@
     )
     (pin "1")
-    (pin "3")
-    (pin "4")
-    (pin "5")
+    (pin "2")
+    (pin "4")
+    (pin "5")
