File: control-board/control-board_v2/control-board_v2.kicad_pcb (KiCad board)
At the start: 4 copper layers, 68.6 x 53.3 mm, 37 parts, among them J1 Barrel_Jack, J2 Header-M_2x6, J3 Header-M_2x6, J4 Header-M_2x6, J5 Header-M_2x6, J6 Header_1x8, J7 Header_1x8, J8 Header_1x10, J9 Header_1x8, Q10 NMOS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

Commit message: drc check fixes
Parts:
- moved R23 0.27 mm to (77.7, 60.4)
Routing:
- net +5V: track 22.3 -> 24.7 mm
- net 3-GND: track 24.1 -> 22.8 mm
Changed lines of the file:
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@@
   )
   (footprint "Resistor_SMD:R_2512_6332Metric" (layer "B.Cu")
-    (at 77.73 60.66 90)
+    (at 77.71 60.39 90)
     (descr "Resistor SMD 2512 (6332 Metric), square (rectangular) end terminal, IPC_7351 nominal, (Body size source: IPC-SM-782 page 72, https://www.pcb-3d.com/wordpress/wp-content/uploads/ipc-sm-782a_amendment_1_and_2.pdf), generated with kicad-footprint-generator")
     (tags "resistor")
@@
   (via (at 41.13 34.91) (size 0.8) (drill 0.4) (layers "F.Cu" "B.Cu") (net 2))
   (via (at 55.52 22.82) (size 0.8) (drill 0.4) (layers "F.Cu" "B.Cu") (net 2))
-  (via (at 78.82 62.38) (size 0.8) (drill 0.4) (layers "F.Cu" "B.Cu") (net 2))
+  (via (at 78.98 61.95) (size 0.8) (drill 0.4) (layers "F.Cu" "B.Cu") (net 2))
   (via (at 27.77 46.04) (size 0.8) (drill 0.4) (layers "F.Cu" "B.Cu") (net 2))
   (via (at 74.52 22.37) (size 0.8) (drill 0.4) (layers "F.Cu" "B.Cu") (net 2))
@@
   (via (at 82.79 46.99) (size 0.8) (drill 0.4) (layers "F.Cu" "B.Cu") (net 2))
   (via (at 59.64 26.52) (size 0.8) (drill 0.4) (layers "F.Cu" "B.Cu") (net 2))
-  (via (at 75.36 63.62) (size 0.8) (drill 0.4) (layers "F.Cu" "B.Cu") (net 2))
+  (via (at 75.33 63.35) (size 0.8) (drill 0.4) (layers "F.Cu" "B.Cu") (net 2))
   (via (at 50.75 22.82) (size 0.8) (drill 0.4) (layers "F.Cu" "B.Cu") (net 2))
   (via (at 55.28 61.97) (size 0.8) (drill 0.4) (layers "F.Cu" "B.Cu") (net 2))
@@
   (via (at 25.08 42.21) (size 0.8) (drill 0.4) (layers "F.Cu" "B.Cu") (net 2))
   (via (at 73.34 20.16) (size 0.8) (drill 0.4) (layers "F.Cu" "B.Cu") (net 2))
+  (segment (start 77.71 63.3525) (end 77.71 63.22) (width 0.25) (layer "B.Cu") (net 2))
   (segment (start 73.3075 22.38) (end 73.3075 20.1925) (width 1) (layer "B.Cu") (net 2))
   (segment (start 55.5125 22.8275) (end 55.52 22.82) (width 0.25) (layer "B.Cu") (net 2))
@@
   (segment (start 74.51 22.38) (end 74.52 22.37) (width 0.25) (layer "B.Cu") (net 2))
   (segment (start 53 22.8275) (end 50.7575 22.8275) (width 1) (layer "B.Cu") (net 2))
+  (segment (start 77.7075 63.35) (end 77.71 63.3525) (width 0.25) (layer "B.Cu") (net 2))
   (segment (start 53 61.9625) (end 50.6375 61.9625) (width 1) (layer "B.Cu") (net 2))
+  (segment (start 77.71 63.22) (end 78.98 61.95) (width 1) (layer "B.Cu") (net 2))
   (segment (start 73.3075 20.1925) (end 73.34 20.16) (width 0.25) (layer "B.Cu") (net 2))
   (segment (start 74.445 44.645) (end 73.65 45.44) (width 0.25) (layer "B.Cu") (net 2))
-  (segment (start 77.73 63.6225) (end 77.73 63.47) (width 0.25) (layer "B.Cu") (net 2))
   (segment (start 50.6375 61.9625) (end 50.63 61.97) (width 1) (layer "B.Cu") (net 2))
-  (segment (start 77.73 63.6225) (end 75.3625 63.6225) (width 1) (layer "B.Cu") (net 2))
-  (segment (start 77.73 63.47) (end 78.82 62.38) (width 1) (layer "B.Cu") (net 2))
   (segment (start 45.67 39.695) (end 45.67 39.07) (width 0.25) (layer "B.Cu") (net 2))
   (segment (start 45.67 39.07) (end 46.3 38.44) (width 0.25) (layer "B.Cu") (net 2))
-  (segment (start 75.3625 63.6225) (end 75.36 63.62) (width 0.25) (layer "B.Cu") (net 2))
+  (segment (start 75.33 63.35) (end 77.7075 63.35) (width 1) (layer "B.Cu") (net 2))
   (segment (start 61.57 25.05) (end 61.57 26.04) (width 0.25) (layer "F.Cu") (net 3))
   (segment (start 44.21 24.86) (end 44.2 24.85) (width 0.25) (layer "F.Cu") (net 3))
@@
   (segment (start 53.27 39.6) (end 53.27 38.97) (width 0.25) (layer "B.Cu") (net 3))
   (segment (start 80.025 39.67) (end 80 39.695) (width 0.25) (layer "B.Cu") (net 3))
+  (segment (start 40.97 46.16) (end 41.86 45.27) (width 0.25) (layer "B.Cu") (net 3))
+  (segment (start 40.42 46.16) (end 40.97 46.16) (width 0.25) (layer "B.Cu") (net 3))
+  (segment (start 41.86 45.27) (end 41.86 44.645) (width 0.25) (layer "B.Cu") (net 3))
   (segment (start 61.800685 26.45) (end 62.58 25.670685) (width 0.25) (layer "B.Cu") (net 3))
   (segment (start 53.27 38.97) (end 52.32 38.02) (width 0.25) (layer "B.Cu") (net 3))
@@
   (segment (start 48.04 39.46) (end 48.04 34.28) (width 1) (layer "F.Cu") (net 5))
   (segment (start 48.04 34.28) (end 49.29 33.03) (width 1) (layer "F.Cu") (net 5))
-  (segment (start 75.52 56.63) (end 75.845 56.955) (width 1) (layer "F.Cu") (net 6))
   (segment (start 75.51 45.01) (end 75.52 45.02) (width 1) (layer "F.Cu") (net 6))
   (segment (start 76.79 58.94) (end 76.79 57.9) (width 0.25) (layer "F.Cu") (net 6))
@@
   (segment (start 75.51 41.2625) (end 75.51 39.81) (width 0.75) (layer "F.Cu") (net 7))
   (segment (start 75.51 34.27) (end 76.79 32.99) (width 1) (layer "F.Cu") (net 7))
-  (segment (start 75.52 39.82) (end 75.51 39.81) (width 1) (layer "F.Cu") (net 7))
   (segment (start 76.79 32.99) (end 76.79 31.94) (width 1) (layer "F.Cu") (net 7))
   (segment (start 75.51 39.81) (end 75.51 34.27) (width 1) (layer "F.Cu") (net 7))
@@
   (segment (start 41.67 53.94) (end 41.61 53.88) (width 0.25) (layer "F.Cu") (net 24))
   (segment (start 69.17 26.89) (end 69.17 20.58) (width 0.25) (layer "F.Cu") (net 24))
+  (segment (start 41.67 20.6645) (end 41.67 26.94) (width 0.25) (layer "F.Cu") (net 24))
   (segment (start 40.73 33.67) (end 40.73 28.89) (width 0.25) (layer "F.Cu") (net 24))
   (segment (start 41.61 39.41) (end 40.2 38) (width 0.25) (layer "F.Cu") (net 24))
@@
   (via (at 41.63 20.6245) (size 0.8) (drill 0.4) (layers "F.Cu" "B.Cu") (net 24))
   (segment (start 42.3845 19.87) (end 41.63 20.6245) (width 0.25) (layer "B.Cu") (net 24))
-  (segment (start 41.67 20.6645) (end 41.67 26.94) (width 0.25) (layer "B.Cu") (net 24))
   (segment (start 68.98 20.39) (end 68.46 19.87) (width 0.25) (layer "B.Cu") (net 24))
   (segment (start 68.46 19.87) (end 42.3845 19.87) (width 0.25) (layer "B.Cu") (net 24))
@@
   (via (at 77.46 46.11) (size 0.8) (drill 0.4) (layers "F.Cu" "B.Cu") (net 65))
   (via (at 77.45 49.15) (size 0.8) (drill 0.4) (layers "F.Cu" "B.Cu") (net 65))
-  (segment (start 76.3275 59.1) (end 77.73 57.6975) (width 0.25) (layer "B.Cu") (net 65))
+  (segment (start 74.27 52.29) (end 77.41 49.15) (width 0.25) (layer "B.Cu") (net 65))
+  (segment (start 77.71 57.4275) (end 77.73 57.4075) (width 1) (layer "B.Cu") (net 65))
   (segment (start 77.46 49.1) (end 77.45 49.11) (width 0.25) (layer "B.Cu") (net 65))
   (segment (start 77.46 44.645) (end 77.46 46.11) (width 0.25) (layer "B.Cu") (net 65))
-  (segment (start 74.27 58.63) (end 74.74 59.1) (width 0.25) (layer "B.Cu") (net 65))
-  (segment (start 74.74 59.1) (end 76.3275 59.1) (width 0.25) (layer "B.Cu") (net 65))
-  (segment (start 74.27 52.29) (end 74.27 58.63) (width 0.25) (layer "B.Cu") (net 65))
-  (segment (start 77.41 49.15) (end 74.27 52.29) (width 0.25) (layer "B.Cu") (net 65))
-  (segment (start 77.73 57.6975) (end 77.73 56.44) (width 1) (layer "B.Cu") (net 65))
-  (segment (start 77.45 49.15) (end 77.41 49.15) (width 0.25) (layer "B.Cu") (net 65))
+  (segment (start 77.73 57.4075) (end 77.73 56.44) (width 1) (layer "B.Cu") (net 65))
+  (segment (start 77.71 57.4275) (end 76.6675 58.47) (width 0.25) (layer "B.Cu") (net 65))
+  (segment (start 76.6675 58.47) (end 75.09 58.47) (width 0.25) (layer "B.Cu") (net 65))
+  (segment (start 75.09 58.47) (end 74.27 57.65) (width 0.25) (layer "B.Cu") (net 65))
+  (segment (start 74.27 57.65) (end 74.27 52.29) (width 0.25) (layer "B.Cu") (net 65))
   (segment (start 77.45 49.11) (end 77.45 49.15) (width 0.25) (layer "B.Cu") (net 65))
+  (segment (start 77.41 49.15) (end 77.45 49.15) (width 0.25) (layer "B.Cu") (net 65))
   (segment (start 79.32 26.9) (end 79.33 26.89) (width 0.25) (layer "F.Cu") (net 66))
   (segment (start 78.07 34.22) (end 78.07 30.03) (width 0.25) (layer "F.Cu") (net 66))

Commit message: control board v2
Parts:
- removed Q10: NMOS, Package_TO_SOT_SMD:SOT-23-6
- removed R24, R42, R47: 0.003, Resistor_SMD:R_2512_6332Metric
- removed R25: 100, Resistor_SMD:R_0805_2012Metric
- removed U6: Opamp_Dual, Package_SO:SOIC-8_3.9x4.9mm_P1.27mm
- added Q2: NMOS, Package_TO_SOT_SMD:SOT-23-6, F.Cu at (73.9, 42.2)
- added R1: 0.003, Resistor_SMD:R_2512_6332Metric, B.Cu at (46.5, 37.0)
- added R10: 10K, Resistor_SMD:R_0805_2012Metric, B.Cu at (41.8, 51.7)
- added R11: 100, Resistor_SMD:R_0805_2012Metric, F.Cu at (41.8, 47.7)
- added R12: 166K, Resistor_SMD:R_0603_1608Metric, B.Cu at (41.8, 47.7)
- added R13: 0.003, Resistor_SMD:R_2512_6332Metric, B.Cu at (75.8, 47.4)
- added R16: 20K, Resistor_SMD:R_0805_2012Metric, B.Cu at (70.7, 49.6)
- added R2: 20K, Resistor_SMD:R_0805_2012Metric, B.Cu at (54.7, 45.4)
- added R29: 166K, Resistor_SMD:R_0603_1608Metric, B.Cu at (70.7, 47.6)
- added R3: 10K, Resistor_SMD:R_0805_2012Metric, B.Cu at (54.7, 49.3)
- added R30: 166K, Resistor_SMD:R_0603_1608Metric, B.Cu at (69.1, 36.8)
- added R4: 20K, Resistor_SMD:R_0805_2012Metric, B.Cu at (40.1, 34.4)
- added R5: 10K, Resistor_SMD:R_0805_2012Metric, B.Cu at (40.1, 32.4)
- added R6: 0.003, Resistor_SMD:R_2512_6332Metric, B.Cu at (47.5, 47.5)
- added R9: 20K, Resistor_SMD:R_0805_2012Metric, B.Cu at (41.8, 49.7)
- added U2: Opamp_Dual, Package_SO:SOIC-8_3.9x4.9mm_P1.27mm, B.Cu at (41.8, 42.2)
- R21: value 100 -> 10K; moved to B.Cu
- R22, R28: value 166K -> 100; footprint Resistor_SMD:R_0603_1608Metric -> Resistor_SMD:R_0805_2012Metric; moved to F.Cu
- R26: value 100 -> 20K; moved to B.Cu
- R27: value 166K -> 10K; footprint Resistor_SMD:R_0603_1608Metric -> Resistor_SMD:R_0805_2012Metric
- moved R21 27.0 mm to (70.7, 51.7), turned to 0 degrees
- moved R22 26.8 mm to (70.7, 47.6)
- moved U4 25.2 mm to (69.0, 42.2), turned to 90 degrees
- moved R23 23.6 mm to (74.6, 37.0), turned to -90 degrees
- moved R26 16.8 mm to (69.1, 34.9)
- moved R28 15.5 mm to (69.1, 36.8), turned to 0 degrees
- moved R27 10.0 mm to (69.1, 32.9), turned to 0 degrees
- moved C3 7.86 mm to (73.7, 37.7), turned to 90 degrees
- moved Q1 4.02 mm to (44.0, 41.6), turned to 0 degrees
- moved C7 2.08 mm to (37.6, 45.7), turned to -90 degrees
- moved R19 1.90 mm to (40.1, 36.4)
- moved R20 1.90 mm to (40.1, 36.4)
- renumbered Q9 to Q1
Connections:
- J2 pad 12: 2-GND -> GND
- J3 pad 12: 1-GND -> GND
- J4 pad 12: 3-GND -> GND
- J5 pad 12: 4-GND -> GND
- J8 pad 1: H1-D12 -> H2-D12
- J8 pad 2: H2-D13 -> H1-D13
- Q1 pad 1: H1-D12 -> H1-D13
- Q1 pad 2: 2-Heater -> GND
- Q1 pad 3: H2-D13 -> H2-D12
- Q1 pad 4: +9V -> 2-Heater
- Q1 pad 5: 1-Heater -> GND
- Q1 pad 6: +9V -> 1-Heater
- R19 pad 1: Net-(U4A--) -> Net-(U2A--)
- R19 pad 2: GND -> Net-(R19-Pad2)
- R20 pad 2: Net-(U4A--) -> Net-(U2A--)
- R21 pad 1: Net-(U4B--) -> Net-(R16-Pad1)
- R22 pad 1: /current-sensing/V_{h2} -> Net-(U4A--)
- R22 pad 2: Net-(U4B--) -> Net-(R16-Pad1)
- R23 pad 1: GND -> 4-Heater
- R23 pad 2: 3-GND -> +9V
- R26 pad 1: Net-(U6A--) -> Net-(R26-Pad1)
- R26 pad 2: GND -> 4-Heater
- R27 pad 1: /current-sensing/V_{h4} -> Net-(R26-Pad1)
- R27 pad 2: Net-(U6B--) -> GND
- R28 pad 1: /current-sensing/V_{h3} -> Net-(U4B--)
- R28 pad 2: Net-(U6A--) -> Net-(R26-Pad1)
- U4 pad 1: /current-sensing/V_{h1} -> /current-sensing/V_{h3}
- U4 pad 3: 1-GND -> Com-Node
- U4 pad 5: 2-GND -> Com-Node
- U4 pad 7: /current-sensing/V_{h2} -> /current-sensing/V_{h4}
Routing:
- net Com-Node: track 0.00 -> 67.3 mm, vias 0 -> 4
- net H1-D12: track 48.5 -> 0.00 mm, vias 2 -> 0
- net H2-D13: track 40.1 -> 0.00 mm
- net ~{RST}: track 99.1 -> 136.2 mm, vias 2 -> 5
- net H2-D12: track 0.00 -> 30.3 mm
- net H1-D13: track 0.00 -> 25.0 mm
- net 2-GND: track 24.6 -> 0.00 mm, vias 3 -> 0
- net 4-GND: track 23.8 -> 0.00 mm, vias 3 -> 0
- net 3-GND: track 22.8 -> 0.00 mm, vias 3 -> 0
- net GND: track 55.6 -> 77.7 mm, vias 26 -> 34
- net 1-CS: track 38.4 -> 60.4 mm, vias 2 -> 4
- net 1-GND: track 21.5 -> 0.00 mm, vias 3 -> 0
- net /current-sensing/V_{h2}: track 45.5 -> 62.2 mm, vias 6 -> 2
- net DIN: track 107.4 -> 121.7 mm, vias 4 -> 5
- net /current-sensing/V_{h1}: track 30.9 -> 43.9 mm, vias 0 -> 2
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
Commit message: v3 with relay
Parts:
- removed C3: 0.1uF, Capacitor_SMD:C_0805_2012Metric
- removed Q1, Q2: NMOS, Package_TO_SOT_SMD:SOT-23-6
- removed R23: 0.003, Resistor_SMD:R_2512_6332Metric
- removed R26: 20K, Resistor_SMD:R_0805_2012Metric
- removed R27: 10K, Resistor_SMD:R_0805_2012Metric
- removed R28: 100, Resistor_SMD:R_0805_2012Metric
- removed R29, R30: 166K, Resistor_SMD:R_0603_1608Metric
- added R14: 0.003, Resistor_SMD:R_2512_6332Metric, B.Cu at (75.5, 36.6)
- added R15: 100, Resistor_SMD:R_0805_2012Metric, B.Cu at (63.7, 35.4)
- added R7: 166K, Resistor_SMD:R_0805_2012Metric, B.Cu at (46.3, 44.7)
- added R8: 166K, Resistor_SMD:R_0805_2012Metric, B.Cu at (41.3, 47.0)
- added U5: LCA701STR, Package_SO:SOIC-6_New, F.Cu at (39.4, 43.2)
- added U6: LCA701STR, Package_SO:SOIC-6_New, F.Cu at (47.8, 41.5)
- added U8: LCA701STR, Package_SO:SOIC-6_New, F.Cu at (71.6, 44.0)
- added U9: LCA701STR, Package_SO:SOIC-6_New, F.Cu at (79.4, 41.8)
- C7, R11, R19: moved to B.Cu
- R10, R3, R5: value 10K -> 100
- R12, R20: footprint Resistor_SMD:R_0603_1608Metric -> Resistor_SMD:R_0805_2012Metric
- R13, R6: value 0.003 -> 166K; footprint Resistor_SMD:R_2512_6332Metric -> Resistor_SMD:R_0805_2012Metric
- R16, R4: value 20K -> 100
- R2, R9: value 20K -> 0.003; footprint Resistor_SMD:R_0805_2012Metric -> Resistor_SMD:R_2512_6332Metric
- R21: value 10K -> 166K
- R22: value 100 -> 166K; moved to B.Cu
- moved R9 33.9 mm to (75.5, 53.4), turned to -90 degrees
- moved R10 23.5 mm to (65.3, 51.5), turned to 180 degrees
- moved R12 19.6 mm to (61.4, 47.0), turned to 180 degrees
- moved R11 19.3 mm to (61.0, 49.4), turned to 0 degrees
- moved R21 17.9 mm to (60.2, 37.1), turned to 180 degrees
- moved R16 17.9 mm to (60.2, 35.1), turned to 180 degrees
- moved R4 13.8 mm to (46.3, 46.7)
- moved R6 13.4 mm to (40.1, 36.4), turned to 0 degrees
- moved R3 13.3 mm to (41.4, 49.6), turned to 180 degrees
- moved R22 12.3 mm to (63.7, 37.4), turned to 180 degrees
- moved R13 10.6 mm to (65.2, 47.1), turned to 180 degrees
- moved R2 8.89 mm to (49.5, 52.6), turned to -90 degrees
- moved U4 5.75 mm to (63.2, 42.2)
- moved R19 3.71 mm to (43.6, 35.1), turned to 0 degrees
- moved R20 3.58 mm to (43.6, 37.1)
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Connections:
- C7 pad 1: +5V -> +9V
- R1 pad 1: 1-Heater -> Net-(R1-Pad1)
- R1 pad 2: +9V -> 1-Heater
- R10 pad 1: Net-(R10-Pad1) -> 3-Heater
- R10 pad 2: GND -> Net-(U4A--)
- R11 pad 1: Net-(U2B--) -> Net-(U4A-+)
- R11 pad 2: Net-(R10-Pad1) -> Net-(R11-Pad2)
- R12 pad 1: /current-sensing/V_{h2} -> Net-(U4A-+)
- R12 pad 2: Net-(U2B--) -> GND
- R13 pad 1: 3-Heater -> /current-sensing/V_{h3}
- R13 pad 2: +9V -> Net-(U4A--)
- R16 pad 1: Net-(R16-Pad1) -> Net-(U4B-+)
- R16 pad 2: 3-Heater -> Net-(R14-Pad1)
- R19 pad 1: Net-(U2A--) -> Net-(U2A-+)
- R19 pad 2: Net-(R19-Pad2) -> Net-(R1-Pad1)
- R2 pad 1: Com-Node -> Net-(R2-Pad1)
- R2 pad 2: +9V -> 2-Heater
- R20 pad 1: /current-sensing/V_{h1} -> Net-(U2A-+)
- R20 pad 2: Net-(U2A--) -> GND
- R21 pad 1: Net-(R16-Pad1) -> Net-(U4B-+)
- R22 pad 1: Net-(U4A--) -> /current-sensing/V_{h4}
- R22 pad 2: Net-(R16-Pad1) -> Net-(U4B--)
- R3 pad 1: Com-Node -> 2-Heater
- R3 pad 2: GND -> Net-(U2B--)
- R4 pad 1: Net-(R19-Pad2) -> Net-(U2B-+)
- R4 pad 2: 1-Heater -> Net-(R2-Pad1)
- R5 pad 1: Net-(R19-Pad2) -> 1-Heater
- R5 pad 2: GND -> Net-(U2A--)
- R6 pad 1: 2-Heater -> /current-sensing/V_{h1}
- R6 pad 2: +9V -> Net-(U2A--)
- R9 pad 1: Net-(R10-Pad1) -> Net-(R11-Pad2)
- R9 pad 2: 2-Heater -> 3-Heater
- U2 pad 3: Com-Node -> Net-(U2A-+)
- U2 pad 5: Com-Node -> Net-(U2B-+)
- U2 pad 8: +5V -> +9V
- U4 pad 3: Com-Node -> Net-(U4A-+)
- U4 pad 5: Com-Node -> Net-(U4B-+)
- U4 pad 8: +5V -> +9V
Routing:
- net Com-Node: track 67.3 -> 0.00 mm, vias 4 -> 0
- net GND: track 77.7 -> 43.7 mm, vias 34 -> 21
- net H2-D12: track 30.3 -> 0.00 mm
- net 2-Heater: track 26.4 -> 1.07 mm, vias 1 -> 0
- net H1-D13: track 25.0 -> 0.00 mm
- net 3-Heater: track 24.3 -> 0.00 mm, vias 1 -> 0
- net 1-Heater: track 20.4 -> 0.00 mm, vias 1 -> 0
- net H4-D19: track 50.8 -> 31.7 mm
- net 4-Heater: track 17.6 -> 0.00 mm, vias 1 -> 0
- net H3-D18: track 71.6 -> 58.5 mm, vias 3 -> 2
- net DOUT: track 129.4 -> 141.3 mm
- net 1-CS_T1: track 22.1 -> 32.4 mm
- net +9V: track 82.4 -> 72.4 mm
- net /current-sensing/V_{h2}: track 62.2 -> 53.5 mm
- net 2-CS: track 29.1 -> 36.8 mm
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Other:
- board text added: "Control Board v3 Boston University N. Gonzalez 10-2024"
- board text removed: "Control Board v2 Boston University N. Gonzalez 08-2024"

Commit message: final layout for controlboard v3
Parts:
- added C3: 0.1uF, Capacitor_SMD:C_0805_2012Metric, B.Cu at (67.8, 38.7)
Connections:
- U5 pad 2: (no net) -> GND
- U5 pad 3: GND -> (no net)
- U6 pad 2: (no net) -> GND
- U6 pad 3: GND -> (no net)
- U8 pad 2: (no net) -> GND
- U8 pad 3: GND -> (no net)
- U9 pad 2: (no net) -> GND
- U9 pad 3: GND -> (no net)
Routing:
- net +9V: track 72.4 -> 131.9 mm, vias 2 -> 10
- net H1-D13: track 0.00 -> 33.6 mm
- net Net-(R14-Pad1): track 0.00 -> 28.4 mm, vias 0 -> 3
- net H4-D19: track 31.7 -> 58.6 mm, vias 1 -> 2
- net GND: track 43.7 -> 70.4 mm, vias 21 -> 31
- net H2-D12: track 0.00 -> 23.6 mm
- net Net-(R11-Pad2): track 0.00 -> 22.8 mm, vias 0 -> 1
- net Net-(R2-Pad1): track 0.00 -> 16.3 mm, vias 0 -> 1
- net 3-Heater: track 0.00 -> 15.8 mm, vias 0 -> 1
- net 2-Heater: track 1.07 -> 16.7 mm, vias 0 -> 3
- net 4-Heater: track 0.00 -> 14.9 mm, vias 0 -> 1
- net Net-(U4A--): track 0.00 -> 10.2 mm, vias 0 -> 2
- net 1-Heater: track 0.00 -> 10.0 mm, vias 0 -> 1
- net Net-(R1-Pad1): track 0.00 -> 9.49 mm, vias 0 -> 1
- net 1-CS_T1: track 32.4 -> 24.0 mm, vias 2 -> 0
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