File: bumpbonds_mockup/hardware/design-files_BM/design-files_BM.kicad_sch (KiCad schematic)
At the start: 42 parts, among them J1 Conn_02x06_Counter_Clockwise, U1 ETROC_bumpbond_dummy, U10 TMP121, U2 ETROC_bumpbond_dummy, U3 ETROC_bumpbond_dummy, U4 ETROC_bumpbond_dummy, U6 ADS7953, U7 TMP121, U8 ADS7953, U9 ADS7953

Commit message: latest TM and BM versions
Parts:
- removed J1: Conn_02x06_Counter_Clockwise, Connector_PinHeader_2.54mm:PinHeader_2x06_P2.54mm_Vertical_SMD, symbol Connector_Generic:Conn_02x06_Counter_Clockwise
- added J2: Conn_02x05_Counter_Clockwise, Connector_PinHeader_2.54mm:PinHeader_2x05_P2.54mm_Vertical_SMD, symbol Connector_Generic:Conn_02x05_Counter_Clockwise
- added R13, R14, R15, R16: 3k3, Resistor_SMD:R_0805_2012Metric_Pad1.20x1.40mm_HandSolder, symbol Device:R
- added TP1, TP10, TP11, TP12, TP13, TP14, TP15, TP16, TP17, TP18, TP19, TP2, TP20, TP21, TP22, TP23, TP24, TP25, TP26, TP27, TP28, TP3, TP4, TP5, TP6, TP7, TP8, TP9: TestPoint, TestPoint:TestPoint_Pad_1.0x1.0mm, symbol Connector:TestPoint
Connections:
- net T1-9 is gone; now on net GND: U1.121 (TP9)
- net +5V: now also J2.4 (Pin_4), R13.2, R14.2, R15.2, R16.2
- net CLK: now also J2.9 (Pin_9)
- net CS_ADC1: now also J2.10 (Pin_10); no longer U6.31 (~{CS}), U8.31 (~{CS})
- net CS_ADC2: now also U6.31 (~{CS}), J2.2 (Pin_2)
- net CS_ADC3: now also U8.31 (~{CS}), J2.1 (Pin_1)
- net CS_T1: now also J2.3 (Pin_3)
- net CS_T2: now also J2.5 (Pin_5)
- net DIN: now also J2.8 (Pin_8)
- net DOUT: now also J2.7 (Pin_7)
- net ETROC1: now also U8.11 (CH15); no longer U9.23 (CH5)
- net ETROC2: now also U6.11 (CH15); no longer U9.21 (CH7)
- net ETROC3: now also U8.25 (CH3); no longer U9.25 (CH3)
- net ETROC4: now also U9.17 (CH9); no longer U9.16 (CH10)
- net GND: now also U2.121 (TP9), U3.121 (TP9), U4.121 (TP9), U6.19 (AGND), U6.20 (AGND), U8.19 (AGND), U8.20 (AGND), U9.10 (AGND), U9.19 (AGND), U9.20 (AGND), J2.6 (Pin_6)
- net LGAD1: now also U8.13 (CH13); no longer U9.24 (CH4)
- net LGAD2: now also U6.13 (CH13); no longer U9.22 (CH6)
- net LGAD3: now also U8.27 (CH1); no longer U9.18 (CH8)
- net LGAD4: now also U9.21 (CH7); no longer U9.17 (CH9)
- net T1-1: now also U8.24 (CH4), R16.1; no longer U6.28 (CH0)
- net T1-2: now also U8.23 (CH5), TP22.1; no longer U6.27 (CH1)
- net T1-3: now also U8.22 (CH6), TP23.1; no longer U6.26 (CH2)
- net T1-4: now also U8.21 (CH7), TP24.1; no longer U6.25 (CH3)
- net T1-5: now also U8.16 (CH10), TP25.1; no longer U6.24 (CH4)
- net T1-6: now also U8.15 (CH11), TP26.1; no longer U6.23 (CH5)
- net T1-7: now also U8.14 (CH12), TP27.1; no longer U6.22 (CH6)
- net T1-8: now also U8.12 (CH14), TP28.1; no longer U6.21 (CH7)
- net T2-1: now also U6.28 (CH0), R15.1; no longer U8.28 (CH0)
- net T2-2: now also U6.27 (CH1), TP15.1; no longer U6.11 (CH15)
- net T2-3: now also U6.26 (CH2), TP16.1; no longer U6.12 (CH14)
- net T2-4: now also U6.25 (CH3), TP17.1; no longer U6.13 (CH13)
- net T2-5: now also U6.16 (CH10), TP18.1; no longer U6.14 (CH12)
- net T2-6: now also TP19.1
- net T2-7: now also U6.14 (CH12), TP20.1; no longer U6.16 (CH10)
- net T2-8: now also U6.12 (CH14), TP21.1; no longer U6.17 (CH9)
- net T3-1: now also U9.16 (CH10), R14.1; no longer U8.27 (CH1)
- net T3-2: now also U9.15 (CH11), TP8.1; no longer U8.26 (CH2)
- net T3-3: now also U9.14 (CH12), TP9.1; no longer U8.25 (CH3)
- net T3-4: now also U9.13 (CH13), TP10.1; no longer U8.24 (CH4)
- net T3-5: now also U9.12 (CH14), TP11.1; no longer U8.23 (CH5)
- net T3-6: now also U9.11 (CH15), TP12.1; no longer U8.22 (CH6)
- net T3-7: now also U8.28 (CH0), TP13.1; no longer U8.21 (CH7)
- net T3-8: now also U8.26 (CH2), TP14.1; no longer U8.18 (CH8)
- net T4-1: now also U9.28 (CH0), R13.1; no longer U8.16 (CH10)
- net T4-2: now also U9.27 (CH1), TP1.1; no longer U8.15 (CH11)
- net T4-3: now also U9.26 (CH2), TP2.1; no longer U8.14 (CH12)
- net T4-4: now also U9.25 (CH3), TP3.1; no longer U8.13 (CH13)
- net T4-5: now also U9.24 (CH4), TP4.1; no longer U8.12 (CH14)
- net T4-6: now also U9.23 (CH5), TP5.1; no longer U8.11 (CH15)
- net T4-7: now also U9.22 (CH6), TP6.1; no longer U9.28 (CH0)
- net T4-8: now also U9.18 (CH8), TP7.1; no longer U9.27 (CH1)
- net at U9.7 (MXO7): now also U9.8 (AINP)
- net at U8.7 (MXO7): now also U8.8 (AINP)
- net at U6.7 (MXO7): now also U6.8 (AINP)
- net T2-9: no longer names the net of U6.18 (CH8)
- net T2-9: no longer U2.121 (TP9)
- net T3-9: no longer names the net of U8.17 (CH9)
- net T3-9: no longer U3.121 (TP9)
- removed net T4-9: U4.121 (TP9), U9.26 (CH2)
- no-connect marks 2 -> 11
Other:
- note added: "Single Resistance: V_{adc} = 5V*R_{adc}/(R_{sel} + R_{adc}) dV_{adc}/dR_{adc} = 5V*R_{sel}/(R_{sel} + R_{adc})^{2} [V/Ω] Maximize the derrivative when R_{sel} = R_{adc} if R_{sel} = 3.3kΩ 0.37 mV/Ω"
- note added: "Voltage Resolution: 5V/ 2^12 = 1.22mV"
- note removed: "CHECK RANGE ASK ABOUT AINP"
- note removed: "Single Resistance: R = 34.6 * T [C] + 9600 Four in Series: R_{ser} = 4*R = 138.4 * T [C] + 38400 V_{sense} = V * (R_{ser} / (R_{ser} + 40k)) -> 4.5mV/[C] near T=0 [C]"
- moved on the sheet: C9
