File: module_pcb_thermal_mockup/hardware/design-files_TM/design-files_TM.kicad_pcb (KiCad board)
At the start: 4 copper layers, 44.1 x 57.5 mm, 59 parts, among them J1 Conn_02x06_Counter_Clockwise, U1 ETROC_dummy_thermal_sensors, U2 ETROC_dummy_thermal_sensors, U3 ETROC_dummy_thermal_sensors, U4 ETROC_dummy_thermal_sensors, U5 AD77x8, U6 AD780, U7 TMP121, U8 TMP121, U9 TMP121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

Commit message: schematic update for more test-points
Other:
- board text added: "ETL Module PCB Thermal Mockup V4 Boston University N. Gonzalez 07-2024"
- board text removed: "locked"

Commit message: files updated
Parts:
- removed 2.5V, TP+, TP-1, TP-2, TP-3, TP-4: TestPoint, TestPoint:TestPoint_Pad_1.0x1.0mm
- removed C1: 1uF, Capacitor_SMD:C_0805_2012Metric_Pad1.18x1.45mm_HandSolder
- removed JMPR1: 0, Resistor_SMD:R_0805_2012Metric_Pad1.20x1.40mm_HandSolder
- removed R13: 1M, Resistor_SMD:R_0805_2012Metric_Pad1.20x1.40mm_HandSolder
- removed RV1: 25k, Potentiometer_SMD:Potentiometer_Bourns_3224W_Vertical
- removed U6: AD780, Package_SO:SOIC-8_3.9x4.9mm_P1.27mm
- added T1:1: TestPoint, TestPoint:TestPoint_Pad_1.0x1.0mm, B.Cu at (1.57, 54.1)
- added T1:2: TestPoint, TestPoint:TestPoint_Pad_1.0x1.0mm, B.Cu at (4.51, 50.5)
- added T1:3: TestPoint, TestPoint:TestPoint_Pad_1.0x1.0mm, B.Cu at (6.60, 50.5)
- added T1:4: TestPoint, TestPoint:TestPoint_Pad_1.0x1.0mm, B.Cu at (12.4, 50.7)
- added T1:5: TestPoint, TestPoint:TestPoint_Pad_1.0x1.0mm, B.Cu at (14.5, 50.7)
- added T1:6: TestPoint, TestPoint:TestPoint_Pad_1.0x1.0mm, B.Cu at (16.6, 50.7)
- added T1:7: TestPoint, TestPoint:TestPoint_Pad_1.0x1.0mm, B.Cu at (18.7, 50.6)
- added T1:8: TestPoint, TestPoint:TestPoint_Pad_1.0x1.0mm, B.Cu at (20.8, 50.6)
- added T1:9: TestPoint, TestPoint:TestPoint_Pad_1.0x1.0mm, B.Cu at (22.9, 50.6)
- added T2:1: TestPoint, TestPoint:TestPoint_Pad_1.0x1.0mm, B.Cu at (25.8, 50.6)
- added T2:2: TestPoint, TestPoint:TestPoint_Pad_1.0x1.0mm, B.Cu at (27.9, 50.6)
- added T2:3: TestPoint, TestPoint:TestPoint_Pad_1.0x1.0mm, B.Cu at (30.0, 50.6)
- added T2:4: TestPoint, TestPoint:TestPoint_Pad_1.0x1.0mm, B.Cu at (32.1, 50.6)
- added T2:5: TestPoint, TestPoint:TestPoint_Pad_1.0x1.0mm, B.Cu at (34.2, 50.6)
- added T2:6: TestPoint, TestPoint:TestPoint_Pad_1.0x1.0mm, B.Cu at (36.3, 50.6)
- added T2:7: TestPoint, TestPoint:TestPoint_Pad_1.0x1.0mm, B.Cu at (38.3, 50.6)
- added T2:8: TestPoint, TestPoint:TestPoint_Pad_1.0x1.0mm, B.Cu at (40.4, 50.6)
- added T2:9: TestPoint, TestPoint:TestPoint_Pad_1.0x1.0mm, B.Cu at (42.5, 50.6)
- added T3:1: TestPoint, TestPoint:TestPoint_Pad_1.0x1.0mm, B.Cu at (18.9, 5.38)
- added T3:2: TestPoint, TestPoint:TestPoint_Pad_1.0x1.0mm, B.Cu at (16.6, 5.39)
- added T3:3: TestPoint, TestPoint:TestPoint_Pad_1.0x1.0mm, B.Cu at (13.6, 5.37)
- added T3:4: TestPoint, TestPoint:TestPoint_Pad_1.0x1.0mm, B.Cu at (11.6, 5.34)
- added T3:5: TestPoint, TestPoint:TestPoint_Pad_1.0x1.0mm, B.Cu at (9.50, 5.35)
- added T3:6: TestPoint, TestPoint:TestPoint_Pad_1.0x1.0mm, B.Cu at (7.43, 5.35)
- added T3:7: TestPoint, TestPoint:TestPoint_Pad_1.0x1.0mm, B.Cu at (5.37, 5.34)
- added T3:8: TestPoint, TestPoint:TestPoint_Pad_1.0x1.0mm, B.Cu at (1.67, 4.48)
- added T3:9: TestPoint, TestPoint:TestPoint_Pad_1.0x1.0mm, B.Cu at (1.67, 1.27)
- added T4:1: TestPoint, TestPoint:TestPoint_Pad_1.0x1.0mm, B.Cu at (40.3, 1.67)
- added T4:2: TestPoint, TestPoint:TestPoint_Pad_1.0x1.0mm, B.Cu at (42.5, 4.95)
- added T4:3: TestPoint, TestPoint:TestPoint_Pad_1.0x1.0mm, B.Cu at (36.3, 6.05)
- added T4:4: TestPoint, TestPoint:TestPoint_Pad_1.0x1.0mm, B.Cu at (34.1, 6.05)
- added T4:5: TestPoint, TestPoint:TestPoint_Pad_1.0x1.0mm, B.Cu at (32.0, 6.06)
- added T4:6: TestPoint, TestPoint:TestPoint_Pad_1.0x1.0mm, B.Cu at (27.5, 5.97)
- added T4:7: TestPoint, TestPoint:TestPoint_Pad_1.0x1.0mm, B.Cu at (25.4, 5.97)
- added T4:8: TestPoint, TestPoint:TestPoint_Pad_1.0x1.0mm, B.Cu at (23.4, 5.97)
- added T4:9: TestPoint, TestPoint:TestPoint_Pad_1.0x1.0mm, B.Cu at (21.2, 5.79)
- U1, U2, U3, U4: value ETROC_dummy_thermal_sensors -> ETROC_bumpbond_dummy; footprint unl_silab:PCB_ETROC2_dummy -> ETL:ETROC2_bumpbonds
- moved C2 24.1 mm to (27.9, 17.0)
- moved C3 17.7 mm to (25.7, 14.9)
- moved C7 1.00 mm to (24.3, 22.5)
- moved E3 1.00 mm to (14.7, 1.70)
- moved E4 1.00 mm to (27.5, 1.70)
- moved L3 1.00 mm to (16.6, 1.70)
- moved L4 1.00 mm to (29.6, 1.70)
Connections:
- R2 pad 2: Net-(JMPR1-Pad1) -> GND
- U1 pad 1: TP+ -> Net-(U1-TP1)
- U2 pad 1: TP+ -> Net-(U2-TP1)
- U3 pad 1: TP+ -> Net-(U3-TP1)
- U4 pad 1: TP+ -> Net-(U4-TP1)
- U5 pad 13: /2.5V -> unconnected-(U5-REFIN2(+)/AIN9-Pad13)
Routing:
- net TP+: track 113.0 -> 0.00 mm, vias 4 -> 0
- net /2.5V: track 32.0 -> 0.00 mm, vias 2 -> 0
- net Net-(JMPR1-Pad1): track 28.2 -> 0.00 mm, vias 4 -> 0
- net /V_{ref}: track 31.4 -> 47.3 mm
- net Net-(U2-TP9): track 9.35 -> 2.82 mm
- net Net-(U1-TP5): track 0.00 -> 5.77 mm, vias 0 -> 1
- net Net-(U1-TP4): track 0.00 -> 5.39 mm, vias 0 -> 1
- net Net-(U3-TP5): track 0.00 -> 4.92 mm, vias 0 -> 1
- net Net-(U1-TP6): track 0.00 -> 4.54 mm, vias 0 -> 1
- net Net-(U4-TP2): track 0.00 -> 4.53 mm, vias 0 -> 1
- net Net-(U2-TP5): track 0.00 -> 4.33 mm, vias 0 -> 1
- net Net-(U2-TP1): track 0.00 -> 4.29 mm, vias 0 -> 1
- net Net-(U4-TP8): track 0.00 -> 4.27 mm, vias 0 -> 1
- net Net-(U1-TP8): track 0.00 -> 4.22 mm, vias 0 -> 1
- net Net-(U4-TP5): track 0.00 -> 4.21 mm, vias 0 -> 1
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Other:
- board text added: "ETL Module PCB Thermal Mockup V4.5 Boston University N. Gonzalez 04-2025"
- board text removed: "ETL Module PCB Thermal Mockup V4 Boston University N. Gonzalez 07-2024"
- board text removed: "Populate for 2.5V on REFIN2"
